Commit message: Adapting model files.

File: Tools/simulation/gz/models/gripper4/gripper4.urdf (robot description, URDF)
Before this commit: robot Assem2_rebuilt, 3 links, 2 joints
Links:
- link base_link: geometry collision mesh filename=package://gripper4/meshes/base_link.STL; visual mesh filename=package://gripper4/meshes/base_link.STL
- link jaw_left: geometry collision mesh filename=package://gripper4/meshes/jaw_left.STL; visual mesh filename=package://gripper4/meshes/jaw_left.STL
- link jaw_right: geometry collision mesh filename=package://gripper4/meshes/jaw_right.STL; visual mesh filename=package://gripper4/meshes/jaw_right.STL
