Commit message: Add the swan_uav_v2 model.

File: Tools/simulation/gz/models/gamma_arm/gamma_arm.urdf (robot description, URDF)
Before this commit: robot GAMMA0, 8 links, 7 joints
Links:
- link A_Link: geometry collision mesh filename=package://gamma_arm/meshes/A_Link.STL; visual mesh filename=package://gamma_arm/meshes/A_Link.STL
- link B_Link: geometry collision mesh filename=package://gamma_arm/meshes/B_Link.STL; visual mesh filename=package://gamma_arm/meshes/B_Link.STL
- link C_Link: geometry collision mesh filename=package://gamma_arm/meshes/C_Link.STL; visual mesh filename=package://gamma_arm/meshes/C_Link.STL
- link D_Link: geometry collision mesh filename=package://gamma_arm/meshes/D_Link.STL; visual mesh filename=package://gamma_arm/meshes/D_Link.STL
- link E_Link: geometry collision mesh filename=package://gamma_arm/meshes/E_Link.STL; visual mesh filename=package://gamma_arm/meshes/E_Link.STL
- link F_Link: geometry collision mesh filename=package://gamma_arm/meshes/F_Link.STL; visual mesh filename=package://gamma_arm/meshes/F_Link.STL
- link base_link: geometry collision mesh filename=package://gamma_arm/meshes/base_link.STL; visual mesh filename=package://gamma_arm/meshes/base_link.STL
