Commit message: Remove original robotic arm from URDF file.

File: Tools/simulation/gz/models/swan_uav_v2/swan_uav_v2.urdf (robot description, URDF)
Before this commit: robot swan_uav_v2, 12 links, 11 joints
Links:
- removed link A_Link
- removed link B_Link
- removed link C_Link
- removed link D_Link
- removed link E_Link
- removed link F_Link
- removed link arm_base_Link
Joints:
- removed joint A_Joint
- removed joint B_Joint
- removed joint C_Joint
- removed joint D_Joint
- removed joint E_Joint
- removed joint F_Joint
- removed joint arm_base_Joint
